Commit message: improved quadrotor model and added PID control to other DOFs
need to tune

File: quadrotor_description/urdf/quadrotor.urdf.xacro (robot description, xacro)
@@ -4,8 +4,14 @@
   <!-- Main properties -->
   <xacro:property name="mass" value="1.477" />
-  <xacro:property name="body_width" value="0.52" />
-  <xacro:property name="body_height" value="0.12" />
-  <xacro:property name="prop_radius" value="0.1" />
-  <xacro:property name="motor_height" value="0.02" />
+  <xacro:property name="body_length" value="0.15" />
+  <xacro:property name="body_width" value="0.15" />
+  <xacro:property name="body_height" value="0.08" />
+  <xacro:property name="arm_length" value="0.25" />
+  <xacro:property name="arm_width" value="0.02" />
+  <xacro:property name="arm_height" value="0.01" />
+  <xacro:property name="prop_radius" value="0.125" />
+  <xacro:property name="prop_height" value="0.005" />
+  <xacro:property name="motor_radius" value="0.015" />
+  <xacro:property name="motor_height" value="0.03" />
   <!-- Colors -->
   <material name="black">
@@ -13,5 +19,5 @@
   </material>
   <material name="blue">
-    <color rgba="0.0 0.0 0.8 1.0"/>
+    <color rgba="0.2 0.2 0.8 1.0"/>
   </material>
   <material name="green">
@@ -21,5 +27,11 @@
     <color rgba="0.8 0.0 0.0 1.0"/>
   </material>
-  <!-- Main quadrotor body -->
+  <material name="gray">
+    <color rgba="0.5 0.5 0.5 1.0"/>
+  </material>
+  <material name="dark_gray">
+    <color rgba="0.3 0.3 0.3 1.0"/>
+  </material>
+  <!-- Main quadrotor body (center) -->
   <link name="base_link">
     <inertial>
@@ -31,5 +43,5 @@
       <origin xyz="0 0 0" rpy="0 0 0" />
       <geometry>
-        <box size="${body_width} ${body_width} ${body_height}"/>
+        <box size="${body_length} ${body_width} ${body_height}"/>
       </geometry>
       <material name="blue"/>
@@ -38,13 +50,39 @@
       <origin xyz="0 0 0" rpy="0 0 0" />
       <geometry>
-        <box size="${body_width} ${body_width} ${body_height}"/>
+        <box size="${body_length} ${body_width} ${body_height}"/>
       </geometry>
     </collision>
   </link>
-  <!-- Rotor links and joints -->
-  <xacro:macro name="rotor" params="name parent x y color">
-    <link name="${name}_link">
-      <inertial>
-        <mass value="0.025" />
+  <!-- Quadrotor arms -->
+  <xacro:macro name="quadrotor_arm" params="name parent x y angle color">
+    <link name="${name}_arm_link">
+      <inertial>
+        <mass value="0.05" />
+        <origin xyz="${arm_length/2} 0 0" />
+        <inertia ixx="0.0001" ixy="0.0" ixz="0.0" iyy="0.001" iyz="0.0" izz="0.001" />
+      </inertial>
+      <visual>
+        <origin xyz="${arm_length/2} 0 0" rpy="0 0 0" />
+        <geometry>
+          <box size="${arm_length} ${arm_width} ${arm_height}"/>
+        </geometry>
+        <material name="dark_gray"/>
+      </visual>
+      <collision>
+        <origin xyz="${arm_length/2} 0 0" rpy="0 0 0" />
+        <geometry>
+          <box size="${arm_length} ${arm_width} ${arm_height}"/>
+        </geometry>
+      </collision>
+    </link>
+    <joint name="${name}_arm_joint" type="fixed">
+      <parent link="${parent}"/>
+      <child link="${name}_arm_link"/>
+      <origin xyz="0 0 0" rpy="0 0 ${angle}"/>
+    </joint>
+    <!-- Motor at the end of the arm -->
+    <link name="${name}_motor_link">
+      <inertial>
+        <mass value="0.03" />
         <origin xyz="0 0 0" />
         <inertia ixx="0.0001" ixy="0.0" ixz="0.0" iyy="0.0001" iyz="0.0" izz="0.0001" />
@@ -53,5 +91,31 @@
         <origin xyz="0 0 0" rpy="0 0 0" />
         <geometry>
-          <cylinder radius="${prop_radius}" length="${motor_height}"/>
+          <cylinder radius="${motor_radius}" length="${motor_height}"/>
+        </geometry>
+        <material name="black"/>
+      </visual>
+      <collision>
+        <origin xyz="0 0 0" rpy="0 0 0" />
+        <geometry>
+          <cylinder radius="${motor_radius}" length="${motor_height}"/>
+        </geometry>
+      </collision>
+    </link>
+    <joint name="${name}_motor_joint" type="fixed">
+      <parent link="${name}_arm_link"/>
+      <child link="${name}_motor_link"/>
+      <origin xyz="${arm_length} 0 ${motor_height/2}" rpy="0 0 0"/>
+    </joint>
+    <!-- Propeller -->
+    <link name="${name}_rotor_link">
+      <inertial>
+        <mass value="0.01" />
+        <origin xyz="0 0 0" />
+        <inertia ixx="0.0001" ixy="0.0" ixz="0.0" iyy="0.0001" iyz="0.0" izz="0.0001" />
+      </inertial>
+      <visual>
+        <origin xyz="0 0 0" rpy="0 0 0" />
+        <geometry>
+          <cylinder radius="${prop_radius}" length="${prop_height}"/>
         </geometry>
         <material name="${color}"/>
@@ -60,19 +124,53 @@
         <origin xyz="0 0 0" rpy="0 0 0" />
         <geometry>
-          <cylinder radius="${prop_radius}" length="${motor_height}"/>
-        </geometry>
-      </collision>
-    </link>
-    <joint name="${name}_joint" type="fixed">
+          <cylinder radius="${prop_radius}" length="${prop_height}"/>
+        </geometry>
+      </collision>
+    </link>
+    <joint name="${name}_rotor_joint" type="continuous">
+      <parent link="${name}_motor_link"/>
+      <child link="${name}_rotor_link"/>
+      <origin xyz="0 0 ${motor_height/2 + prop_height/2}" rpy="0 0 0"/>
+      <axis xyz="0 0 1"/>
+    </joint>
+  </xacro:macro>
+  <!-- Create four arms with rotors -->
+  <xacro:quadrotor_arm name="front_right" parent="base_link" x="1" y="-1" angle="${pi/4}" color="green"/>
+  <xacro:quadrotor_arm name="front_left" parent="base_link" x="1" y="1" angle="${3*pi/4}" color="green"/>
+  <xacro:quadrotor_arm name="back_right" parent="base_link" x="-1" y="-1" angle="${-pi/4}" color="red"/>
+  <xacro:quadrotor_arm name="back_left" parent="base_link" x="-1" y="1" angle="${-3*pi/4}" color="red"/>
+  <!-- Landing gear -->
+  <xacro:macro name="landing_leg" params="name parent x y">
+    <link name="${name}_leg_link">
+      <inertial>
+        <mass value="0.01" />
+        <origin xyz="0 0 -0.05" />
+        <inertia ixx="0.0001" ixy="0.0" ixz="0.0" iyy="0.0001" iyz="0.0" izz="0.0001" />
+      </inertial>
+      <visual>
+        <origin xyz="0 0 -0.05" rpy="0 0 0" />
+        <geometry>
+          <cylinder radius="0.005" length="0.1"/>
+        </geometry>
+        <material name="black"/>
+      </visual>
+      <collision>
+        <origin xyz="0 0 -0.05" rpy="0 0 0" />
+        <geometry>
+          <cylinder radius="0.005" length="0.1"/>
+        </geometry>
+      </collision>
+    </link>
+    <joint name="${name}_leg_joint" type="fixed">
       <parent link="${parent}"/>
-      <child link="${name}_link"/>
-      <origin xyz="${x} ${y} 0" rpy="0 0 0"/>
+      <child link="${name}_leg_link"/>
+      <origin xyz="${x*0.08} ${y*0.08} -${body_height/2}" rpy="0 0 0"/>
     </joint>
   </xacro:macro>
-  <!-- Create rotors -->
-  <xacro:rotor name="front_right_rotor" parent="base_link" x="${body_width/3}" y="-${body_width/3}" color="green"/>
-  <xacro:rotor name="front_left_rotor" parent="base_link" x="${body_width/3}" y="${body_width/3}" color="green"/>
-  <xacro:rotor name="back_right_rotor" parent="base_link" x="-${body_width/3}" y="-${body_width/3}" color="red"/>
-  <xacro:rotor name="back_left_rotor" parent="base_link" x="-${body_width/3}" y="${body_width/3}" color="red"/>
+  <!-- Create landing legs -->
+  <xacro:landing_leg name="front_right" parent="base_link" x="1" y="-1"/>
+  <xacro:landing_leg name="front_left" parent="base_link" x="1" y="1"/>
+  <xacro:landing_leg name="back_right" parent="base_link" x="-1" y="-1"/>
+  <xacro:landing_leg name="back_left" parent="base_link" x="-1" y="1"/>
   <!-- Bottom camera -->
   <link name="bottom_camera_link">
@@ -85,5 +183,5 @@
       <origin xyz="0 0 0" rpy="0 0 0" />
       <geometry>
-        <box size="0.05 0.05 0.05"/>
+        <box size="0.03 0.03 0.02"/>
       </geometry>
       <material name="black"/>
@@ -92,5 +190,5 @@
       <origin xyz="0 0 0" rpy="0 0 0" />
       <geometry>
-        <box size="0.05 0.05 0.05"/>
+        <box size="0.03 0.03 0.02"/>
       </geometry>
     </collision>
@@ -99,17 +197,17 @@
     <parent link="base_link"/>
     <child link="bottom_camera_link"/>
-    <origin xyz="0 0 -${body_height/2 + 0.025}" rpy="0 ${pi/2} 0"/>
+    <origin xyz="0 0 -${body_height/2 + 0.01}" rpy="0 ${pi/2} 0"/>
   </joint>
   <!-- IMU Link -->
   <link name="imu_link">
     <inertial>
-      <mass value="0.01" />
-      <origin xyz="0 0 0" />
-      <inertia ixx="0.0001" ixy="0.0" ixz="0.0" iyy="0.0001" iyz="0.0" izz="0.0001" />
-    </inertial>
-    <visual>
-      <origin xyz="0 0 0" rpy="0 0 0" />
-      <geometry>
-        <box size="0.02 0.02 0.02"/>
+      <mass value="0.005" />
+      <origin xyz="0 0 0" />
+      <inertia ixx="0.00001" ixy="0.0" ixz="0.0" iyy="0.00001" iyz="0.0" izz="0.00001" />
+    </inertial>
+    <visual>
+      <origin xyz="0 0 0" rpy="0 0 0" />
+      <geometry>
+        <box size="0.015 0.015 0.005"/>
       </geometry>
       <material name="red"/>
@@ -124,12 +222,12 @@
   <link name="gps_link">
     <inertial>
-      <mass value="0.01" />
-      <origin xyz="0 0 0" />
-      <inertia ixx="0.0001" ixy="0.0" ixz="0.0" iyy="0.0001" iyz="0.0" izz="0.0001" />
-    </inertial>
-    <visual>
-      <origin xyz="0 0 0" rpy="0 0 0" />
-      <geometry>
-        <cylinder radius="0.02" length="0.02"/>
+      <mass value="0.005" />
+      <origin xyz="0 0 0" />
+      <inertia ixx="0.00001" ixy="0.0" ixz="0.0" iyy="0.00001" iyz="0.0" izz="0.00001" />
+    </inertial>
+    <visual>
+      <origin xyz="0 0 0" rpy="0 0 0" />
+      <geometry>
+        <cylinder radius="0.015" length="0.005"/>
       </geometry>
       <material name="black"/>
@@ -139,5 +237,5 @@
     <parent link="base_link"/>
     <child link="gps_link"/>
-    <origin xyz="0 0 ${body_height/2 + 0.01}" rpy="0 0 0"/>
+    <origin xyz="0 0 ${body_height/2 + 0.0025}" rpy="0 0 0"/>
   </joint>
 </robot>

Commit message: cleaned up urdf

File: quadrotor_description/urdf/quadrotor.urdf.xacro (robot description, xacro)
@@ -14,23 +14,23 @@
   <xacro:property name="motor_radius" value="0.015" />
   <xacro:property name="motor_height" value="0.03" />
-  <!-- Colors -->
+  <!-- Updated Colors for cleaner look -->
   <material name="black">
     <color rgba="0.0 0.0 0.0 1.0"/>
   </material>
-  <material name="blue">
-    <color rgba="0.2 0.2 0.8 1.0"/>
-  </material>
-  <material name="green">
-    <color rgba="0.0 0.8 0.0 1.0"/>
-  </material>
-  <material name="red">
-    <color rgba="0.8 0.0 0.0 1.0"/>
-  </material>
-  <material name="gray">
-    <color rgba="0.5 0.5 0.5 1.0"/>
+  <material name="white">
+    <color rgba="1.0 1.0 1.0 1.0"/>
+  </material>
+  <material name="light_gray">
+    <color rgba="0.7 0.7 0.7 1.0"/>
   </material>
   <material name="dark_gray">
     <color rgba="0.3 0.3 0.3 1.0"/>
   </material>
+  <material name="blue">
+    <color rgba="0.1 0.5 0.69 1.0"/>
+  </material>
+  <material name="green">
+    <color rgba="0.1 0.69 0.5 1.0"/>
+  </material>
   <!-- Main quadrotor body (center) -->
   <link name="base_link">
@@ -45,5 +45,5 @@
         <box size="${body_length} ${body_width} ${body_height}"/>
       </geometry>
-      <material name="blue"/>
+      <material name="white"/>
     </visual>
     <collision>
@@ -136,8 +136,8 @@
   </xacro:macro>
   <!-- Create four arms with rotors -->
-  <xacro:quadrotor_arm name="front_right" parent="base_link" x="1" y="-1" angle="${pi/4}" color="green"/>
-  <xacro:quadrotor_arm name="front_left" parent="base_link" x="1" y="1" angle="${3*pi/4}" color="green"/>
-  <xacro:quadrotor_arm name="back_right" parent="base_link" x="-1" y="-1" angle="${-pi/4}" color="red"/>
-  <xacro:quadrotor_arm name="back_left" parent="base_link" x="-1" y="1" angle="${-3*pi/4}" color="red"/>
+  <xacro:quadrotor_arm name="front_right" parent="base_link" x="1" y="-1" angle="${pi/4}" color="blue"/>
+  <xacro:quadrotor_arm name="front_left" parent="base_link" x="1" y="1" angle="${3*pi/4}" color="blue"/>
+  <xacro:quadrotor_arm name="back_left" parent="base_link" x="-1" y="1" angle="${-3*pi/4}" color="green"/>
+  <xacro:quadrotor_arm name="back_right" parent="base_link" x="-1" y="-1" angle="${-pi/4}" color="green"/>
   <!-- Landing gear -->
   <xacro:macro name="landing_leg" params="name parent x y">
@@ -171,6 +171,6 @@
   <xacro:landing_leg name="front_right" parent="base_link" x="1" y="-1"/>
   <xacro:landing_leg name="front_left" parent="base_link" x="1" y="1"/>
+  <xacro:landing_leg name="back_left" parent="base_link" x="-1" y="1"/>
   <xacro:landing_leg name="back_right" parent="base_link" x="-1" y="-1"/>
-  <xacro:landing_leg name="back_left" parent="base_link" x="-1" y="1"/>
   <!-- Bottom camera -->
   <link name="bottom_camera_link">
@@ -211,5 +211,5 @@
         <box size="0.015 0.015 0.005"/>
       </geometry>
-      <material name="red"/>
+      <material name="light_gray"/>
     </visual>
   </link>
@@ -231,5 +231,5 @@
         <cylinder radius="0.015" length="0.005"/>
       </geometry>
-      <material name="black"/>
+      <material name="light_gray"/>
     </visual>
   </link>
