Commit message: modified platform dimensions and spawn position and drone behaviour to land on the platform

File: quadrotor_description/urdf/platform/platform.urdf.xacro (robot description, xacro)
@@ -2,14 +2,14 @@
 <robot name="platform" xmlns:xacro="http://www.ros.org/wiki/xacro">
   <!-- Platform dimensions -->
-  <xacro:property name="platform_length" value="1.5" />
-  <xacro:property name="platform_width" value="1.5" />
-  <xacro:property name="platform_height" value="0.5" />
-  <xacro:property name="marker_size" value="1.0" />
+  <xacro:property name="platform_length" value="1.0" />
+  <xacro:property name="platform_width" value="1.0" />
+  <xacro:property name="platform_height" value="0.2" />
+  <xacro:property name="marker_size" value="0.8" />
   <!-- Base link -->
   <link name="base_link">
     <inertial>
       <origin xyz="0 0 0" rpy="0 0 0"/>
-      <mass value="50.0"/>
-      <inertia ixx="9.375" ixy="0.0" ixz="0.0" iyy="9.375" iyz="0.0" izz="18.75"/>
+      <mass value="20.0"/>
+      <inertia ixx="1.67" ixy="0.0" ixz="0.0" iyy="1.67" iyz="0.0" izz="3.33"/>
     </inertial>
     <visual>
@@ -66,5 +66,5 @@
     <parent link="base_link"/>
     <child link="gps_link"/>
-    <origin xyz="0.6 0.6 ${platform_height/2 + 0.01}" rpy="0 0 0"/>
+    <origin xyz="0.45 0.45 ${platform_height/2 + 0.01}" rpy="0 0 0"/>
   </joint>
 </robot>
