Commit message: rotated camera to fix orientation bug

File: quadrotor_description/models/quadrotor/quadrotor.urdf.xacro (robot description, xacro)
@@ -197,5 +197,5 @@
     <parent link="base_link"/>
     <child link="bottom_camera_link"/>
-    <origin xyz="0 0 -${body_height/2 + 0.01}" rpy="0 ${pi/2} 0"/>
+    <origin xyz="0 0 -${body_height/2 + 0.01}" rpy="0 ${pi/2} ${pi/2}"/>
   </joint>
   <!-- IMU Link -->
