Commit message: minor changes

File: quadrotor_description/models/platform/platform.urdf.xacro (robot description, xacro)
@@ -1,4 +1,5 @@
 <?xml version="1.0"?>
 <robot name="platform" xmlns:xacro="http://www.ros.org/wiki/xacro">
+  <xacro:property name="pi" value="3.1415926535897931" />
   <!-- Platform dimensions -->
   <xacro:property name="platform_length" value="1.0" />
